File: pcb/V2/dxhubV2.kicad_pcb (KiCad board)
At the start: 2 copper layers, 75 x 75 mm, 8 parts, among them SW2 MSK12C02, U1 XL-3210SYGC, U2 XL-3210SYGC, U3 XL-3210SYGC

Commit message: New NF, Noyce, and DXHub logo; cleaned up copper fills on back; reversed LEDs to match datasheet
Parts:
- added G***: LOGO, LOGO, B.Cu at (46.6, 28.4)
