File: pcb/V2/dxhubV2.kicad_sch (KiCad schematic)
At the start: 8 parts, among them SW2 MSK12C02, U1 XL-3210SYGC, U2 XL-3210SYGC, U3 XL-3210SYGC

Commit message: New NF, Noyce, and DXHub logo; cleaned up copper fills on back; reversed LEDs to match datasheet
Parts:
- R1, R2, R3: value 1206W4J0390T5E -> 40R
- renumbered U1 to LED1, U2 to LED2, U3 to LED3
Connections:
- net GND: no longer LED1.3, LED2.3, LED3.3
- net at R1.2: now also LED1.2; no longer LED1.1
- net at LED3.1: now also LED1.1, LED2.1, SW2.2; no longer R3.2
- net at R2.2: now also LED2.2; no longer LED2.1
- new net: LED3.2, R3.2
